Commit message: MVP-01 단위 테스트 및 패키지 테스트 확인.

File: ros2_ws/src/safe_drive_description/urdf/ego_vehicle.urdf.xacro (robot description, xacro)
@@ -1,76 +1,5 @@
 <?xml version="1.0"?>
 <robot name="safe_drive_ego" xmlns:xacro="http://www.ros.org/wiki/xacro">
-  <!--
-    A deliberately simple vehicle model for MVP-01.  Its geometry is kept in
-    this file so later Gazebo plugins and controllers can share one definition.
-  -->
-  <xacro:property name="chassis_length" value="0.90"/>
-  <xacro:property name="chassis_width" value="0.50"/>
-  <xacro:property name="chassis_height" value="0.20"/>
-  <xacro:property name="wheel_radius" value="0.10"/>
-  <xacro:property name="wheel_width" value="0.06"/>
-  <material name="blue">
-    <color rgba="0.10 0.35 0.80 1.0"/>
-  </material>
-  <material name="black">
-    <color rgba="0.05 0.05 0.05 1.0"/>
-  </material>
-  <link name="base_footprint"/>
-  <joint name="base_footprint_joint" type="fixed">
-    <parent link="base_footprint"/>
-    <child link="base_link"/>
-    <origin xyz="0 0 0.25" rpy="0 0 0"/>
-  </joint>
-  <link name="base_link">
-    <inertial>
-      <origin xyz="0 0 0" rpy="0 0 0"/>
-      <mass value="12.0"/>
-      <inertia ixx="0.32" ixy="0.0" ixz="0.0" iyy="0.92" iyz="0.0" izz="1.12"/>
-    </inertial>
-    <visual>
-      <origin xyz="0 0 0" rpy="0 0 0"/>
-      <geometry>
-        <box size="${chassis_length} ${chassis_width} ${chassis_height}"/>
-      </geometry>
-      <material name="blue"/>
-    </visual>
-    <collision>
-      <origin xyz="0 0 0" rpy="0 0 0"/>
-      <geometry>
-        <box size="${chassis_length} ${chassis_width} ${chassis_height}"/>
-      </geometry>
-    </collision>
-  </link>
-  <xacro:macro name="wheel" params="name x y">
-    <link name="${name}">
-      <inertial>
-        <origin xyz="0 0 0" rpy="0 0 0"/>
-        <mass value="0.5"/>
-        <inertia ixx="0.0028" ixy="0.0" ixz="0.0" iyy="0.0025" iyz="0.0" izz="0.0028"/>
-      </inertial>
-      <visual>
-        <origin xyz="0 0 0" rpy="1.57079632679 0 0"/>
-        <geometry>
-          <cylinder radius="${wheel_radius}" length="${wheel_width}"/>
-        </geometry>
-        <material name="black"/>
-      </visual>
-      <collision>
-        <origin xyz="0 0 0" rpy="1.57079632679 0 0"/>
-        <geometry>
-          <cylinder radius="${wheel_radius}" length="${wheel_width}"/>
-        </geometry>
-      </collision>
-    </link>
-    <joint name="${name}_joint" type="continuous">
-      <parent link="base_link"/>
-      <child link="${name}"/>
-      <origin xyz="${x} ${y} -0.15" rpy="0 0 0"/>
-      <axis xyz="0 1 0"/>
-    </joint>
-  </xacro:macro>
-  <xacro:wheel name="front_left_wheel" x="0.30" y="0.28"/>
-  <xacro:wheel name="front_right_wheel" x="0.30" y="-0.28"/>
-  <xacro:wheel name="rear_left_wheel" x="-0.30" y="0.28"/>
-  <xacro:wheel name="rear_right_wheel" x="-0.30" y="-0.28"/>
+  <xacro:include filename="$(find safe_drive_description)/urdf/ego_vehicle_core.xacro"/>
+  <xacro:safe_drive_ego_vehicle/>
 </robot>
