Commit message: Build integrated traffic scene and signal control

File: ros2_ws/src/safe_drive_description/urdf/ego_vehicle_core.xacro (robot description, xacro)
@@ -2,10 +2,10 @@
 <robot xmlns:xacro="http://www.ros.org/wiki/xacro">
   <!-- Simulator-independent geometry shared by the plain and Gazebo models. -->
-  <xacro:macro name="safe_drive_ego_vehicle" params="">
-    <xacro:property name="chassis_length" value="0.90"/>
-    <xacro:property name="chassis_width" value="0.50"/>
-    <xacro:property name="chassis_height" value="0.20"/>
-    <xacro:property name="wheel_radius" value="0.10"/>
-    <xacro:property name="wheel_width" value="0.06"/>
+  <xacro:macro name="safe_drive_ego_vehicle" params="use_reference_mesh:=true">
+    <xacro:property name="chassis_length" value="4.20"/>
+    <xacro:property name="chassis_width" value="1.80"/>
+    <xacro:property name="chassis_height" value="1.20"/>
+    <xacro:property name="wheel_radius" value="0.30"/>
+    <xacro:property name="wheel_width" value="0.18"/>
     <material name="blue">
       <color rgba="0.10 0.35 0.80 1.0"/>
@@ -14,23 +14,137 @@
       <color rgba="0.05 0.05 0.05 1.0"/>
     </material>
+    <material name="glass">
+      <color rgba="0.13 0.22 0.28 1.0"/>
+    </material>
+    <material name="lamp">
+      <color rgba="0.92 0.91 0.78 1.0"/>
+    </material>
+    <material name="paint_highlight"><color rgba="0.20 0.55 0.88 1"/></material>
+    <material name="dark_trim"><color rgba="0.025 0.035 0.045 1"/></material>
+    <material name="silver"><color rgba="0.57 0.64 0.69 1"/></material>
+    <material name="tail_lamp"><color rgba="0.82 0.055 0.035 1"/></material>
     <link name="base_footprint"/>
     <joint name="base_footprint_joint" type="fixed">
       <parent link="base_footprint"/>
       <child link="base_link"/>
-      <origin xyz="0 0 0.25" rpy="0 0 0"/>
+      <origin xyz="0 0 0.75" rpy="0 0 0"/>
     </joint>
     <link name="base_link">
       <inertial>
         <origin xyz="0 0 0" rpy="0 0 0"/>
-        <mass value="12.0"/>
-        <inertia ixx="0.32" ixy="0.0" ixz="0.0" iyy="0.92" iyz="0.0" izz="1.12"/>
+        <mass value="120.0"/>
+        <inertia ixx="30.6" ixy="0.0" ixz="0.0" iyy="158.8" iyz="0.0" izz="187.2"/>
       </inertial>
-      <visual>
-        <origin xyz="0 0 0" rpy="0 0 0"/>
+      <!-- The Prius exterior is from osrf/car_demo. Keep the SAFE-Drive
+           collision and dynamics independent of its visual mesh. -->
+      <xacro:if value="${use_reference_mesh}">
+        <visual name="prius_body">
+          <origin xyz="0 0 -0.75" rpy="0 0 1.57079632679"/>
+          <geometry>
+            <mesh filename="file://$(find safe_drive_description)/meshes/prius/hybrid_body.obj"
+                  scale="0.009 0.009 0.01"/>
+          </geometry>
+        </visual>
+      </xacro:if>
+      <xacro:unless value="${use_reference_mesh}">
+      <!-- Earlier primitive exterior remains available for asset diagnosis. -->
+      <visual name="lower_body">
+        <origin xyz="0 0 -0.12" rpy="0 0 0"/>
         <geometry>
-          <box size="${chassis_length} ${chassis_width} ${chassis_height}"/>
+          <box size="${chassis_length} ${chassis_width} 0.70"/>
         </geometry>
         <material name="blue"/>
       </visual>
+      <visual name="body_shoulder">
+        <origin xyz="0 0 0.19" rpy="0 0 0"/>
+        <geometry><box size="4.08 1.76 0.20"/></geometry>
+        <material name="paint_highlight"/>
+      </visual>
+      <visual name="cabin_glass">
+        <origin xyz="-0.30 0 0.49" rpy="0 0 0"/>
+        <geometry><box size="2.15 1.49 0.50"/></geometry>
+        <material name="glass"/>
+      </visual>
+      <visual name="roof">
+        <origin xyz="-0.36 0 0.79" rpy="0 0 0"/>
+        <geometry><box size="1.70 1.52 0.10"/></geometry>
+        <material name="blue"/>
+      </visual>
+      <visual name="front_pillar">
+        <origin xyz="0.73 0 0.54" rpy="0 -0.40 0"/>
+        <geometry><box size="0.10 1.53 0.56"/></geometry>
+        <material name="blue"/>
+      </visual>
+      <visual name="rear_pillar">
+        <origin xyz="-1.30 0 0.54" rpy="0 0.43 0"/>
+        <geometry><box size="0.10 1.53 0.56"/></geometry>
+        <material name="blue"/>
+      </visual>
+      <visual name="left_center_pillar">
+        <origin xyz="-0.30 0.755 0.49" rpy="0 0 0"/>
+        <geometry><box size="0.09 0.035 0.50"/></geometry>
+        <material name="dark_trim"/>
+      </visual>
+      <visual name="right_center_pillar">
+        <origin xyz="-0.30 -0.755 0.49" rpy="0 0 0"/>
+        <geometry><box size="0.09 0.035 0.50"/></geometry>
+        <material name="dark_trim"/>
+      </visual>
+      <visual name="left_side_sill">
+        <origin xyz="0 0.906 -0.36" rpy="0 0 0"/>
+        <geometry><box size="2.45 0.028 0.08"/></geometry>
+        <material name="dark_trim"/>
+      </visual>
+      <visual name="right_side_sill">
+        <origin xyz="0 -0.906 -0.36" rpy="0 0 0"/>
+        <geometry><box size="2.45 0.028 0.08"/></geometry>
+        <material name="dark_trim"/>
+      </visual>
+      <visual name="front_grille">
+        <origin xyz="2.106 0 -0.16" rpy="0 0 0"/>
+        <geometry><box size="0.014 0.83 0.19"/></geometry>
+        <material name="dark_trim"/>
+      </visual>
+      <visual name="front_bumper">
+        <origin xyz="2.10 0 -0.37" rpy="0 0 0"/>
+        <geometry><box size="0.12 1.70 0.13"/></geometry>
+        <material name="dark_trim"/>
+      </visual>
+      <visual name="rear_bumper">
+        <origin xyz="-2.10 0 -0.37" rpy="0 0 0"/>
+        <geometry><box size="0.12 1.70 0.13"/></geometry>
+        <material name="dark_trim"/>
+      </visual>
+      <visual name="front_left_headlamp">
+        <origin xyz="2.106 0.65 0.06" rpy="0 0 0"/>
+        <geometry><box size="0.014 0.35 0.14"/></geometry>
+        <material name="lamp"/>
+      </visual>
+      <visual name="front_right_headlamp">
+        <origin xyz="2.106 -0.65 0.06" rpy="0 0 0"/>
+        <geometry><box size="0.014 0.35 0.14"/></geometry>
+        <material name="lamp"/>
+      </visual>
+      <visual name="rear_left_lamp">
+        <origin xyz="-2.106 0.65 0.06" rpy="0 0 0"/>
+        <geometry><box size="0.014 0.35 0.14"/></geometry>
+        <material name="tail_lamp"/>
+      </visual>
+      <visual name="rear_right_lamp">
+        <origin xyz="-2.106 -0.65 0.06" rpy="0 0 0"/>
+        <geometry><box size="0.014 0.35 0.14"/></geometry>
+        <material name="tail_lamp"/>
+      </visual>
+      <visual name="left_mirror">
+        <origin xyz="0.66 0.96 0.36" rpy="0 0 0"/>
+        <geometry><box size="0.27 0.15 0.13"/></geometry>
+        <material name="dark_trim"/>
+      </visual>
+      <visual name="right_mirror">
+        <origin xyz="0.66 -0.96 0.36" rpy="0 0 0"/>
+        <geometry><box size="0.27 0.15 0.13"/></geometry>
+        <material name="dark_trim"/>
+      </visual>
+      </xacro:unless>
       <collision>
         <origin xyz="0 0 0" rpy="0 0 0"/>
@@ -40,18 +154,37 @@
       </collision>
     </link>
-    <xacro:macro name="wheel" params="name x y">
+    <xacro:macro name="wheel" params="name x y side">
       <link name="${name}">
         <inertial>
           <origin xyz="0 0 0" rpy="0 0 0"/>
-          <mass value="0.5"/>
-          <inertia ixx="0.0028" ixy="0.0" ixz="0.0" iyy="0.0025" iyz="0.0" izz="0.0028"/>
+          <mass value="2.0"/>
+          <inertia ixx="0.05" ixy="0.0" ixz="0.0" iyy="0.09" iyz="0.0" izz="0.05"/>
         </inertial>
-        <visual>
-          <origin xyz="0 0 0" rpy="1.57079632679 0 0"/>
-          <geometry>
-            <cylinder radius="${wheel_radius}" length="${wheel_width}"/>
-          </geometry>
-          <material name="black"/>
-        </visual>
+        <xacro:if value="${use_reference_mesh}">
+          <visual name="prius_wheel">
+            <origin xyz="0 0 0" rpy="0 0 1.57079632679"/>
+            <geometry>
+              <mesh filename="file://$(find safe_drive_description)/meshes/prius/wheel.obj"
+                    scale="0.01 0.01 0.01"/>
+            </geometry>
+          </visual>
+        </xacro:if>
+        <xacro:unless value="${use_reference_mesh}">
+          <visual name="tire">
+            <origin xyz="0 0 0" rpy="1.57079632679 0 0"/>
+            <geometry><cylinder radius="${wheel_radius}" length="${wheel_width}"/></geometry>
+            <material name="black"/>
+          </visual>
+          <visual name="outer_hub">
+            <origin xyz="0 ${0.095 * side} 0" rpy="1.57079632679 0 0"/>
+            <geometry><cylinder radius="0.17" length="0.012"/></geometry>
+            <material name="silver"/>
+          </visual>
+          <visual name="hub_center">
+            <origin xyz="0 ${0.103 * side} 0" rpy="1.57079632679 0 0"/>
+            <geometry><cylinder radius="0.055" length="0.013"/></geometry>
+            <material name="dark_trim"/>
+          </visual>
+        </xacro:unless>
         <collision>
           <origin xyz="0 0 0" rpy="1.57079632679 0 0"/>
@@ -64,13 +197,13 @@
         <parent link="base_link"/>
         <child link="${name}"/>
-        <origin xyz="${x} ${y} -0.15" rpy="0 0 0"/>
+        <origin xyz="${x} ${y} -0.45" rpy="0 0 0"/>
         <axis xyz="0 1 0"/>
         <dynamics damping="0.1" friction="0.0"/>
       </joint>
     </xacro:macro>
-    <xacro:wheel name="front_left_wheel" x="0.30" y="0.28"/>
-    <xacro:wheel name="front_right_wheel" x="0.30" y="-0.28"/>
-    <xacro:wheel name="rear_left_wheel" x="-0.30" y="0.28"/>
-    <xacro:wheel name="rear_right_wheel" x="-0.30" y="-0.28"/>
+    <xacro:wheel name="front_left_wheel" x="1.25" y="0.78" side="1"/>
+    <xacro:wheel name="front_right_wheel" x="1.25" y="-0.78" side="-1"/>
+    <xacro:wheel name="rear_left_wheel" x="-1.25" y="0.78" side="1"/>
+    <xacro:wheel name="rear_right_wheel" x="-1.25" y="-0.78" side="-1"/>
   </xacro:macro>
 </robot>

File: ros2_ws/src/safe_drive_sim/urdf/ego_vehicle.gazebo.urdf.xacro (robot description, xacro)
@@ -20,4 +20,17 @@
   <xacro:wheel_surface name="rear_left_wheel"/>
   <xacro:wheel_surface name="rear_right_wheel"/>
+  <gazebo reference="base_footprint">
+    <sensor type="contact" name="pedestrian_contact">
+      <update_rate>60</update_rate>
+      <contact><collision>base_footprint_fixed_joint_lump__base_link_collision</collision></contact>
+      <plugin name="safe_drive_contact" filename="libgazebo_ros_bumper.so">
+        <ros>
+          <namespace>/safe_drive/ego</namespace>
+          <remapping>bumper_states:=contacts</remapping>
+        </ros>
+        <frame_name>base_link</frame_name>
+      </plugin>
+    </sensor>
+  </gazebo>
   <!-- Four-wheel skid-steer drive keeps the MVP deterministic and exposes the
        standard Twist/Odometry interface needed by the waypoint controller. -->
@@ -33,10 +46,10 @@
       <left_joint>rear_left_wheel_joint</left_joint>
       <right_joint>rear_right_wheel_joint</right_joint>
-      <wheel_separation>0.56</wheel_separation>
-      <wheel_separation>0.56</wheel_separation>
-      <wheel_diameter>0.20</wheel_diameter>
-      <wheel_diameter>0.20</wheel_diameter>
-      <max_wheel_torque>10.0</max_wheel_torque>
-      <max_wheel_acceleration>2.0</max_wheel_acceleration>
+      <wheel_separation>1.56</wheel_separation>
+      <wheel_separation>1.56</wheel_separation>
+      <wheel_diameter>0.60</wheel_diameter>
+      <wheel_diameter>0.60</wheel_diameter>
+      <max_wheel_torque>100.0</max_wheel_torque>
+      <max_wheel_acceleration>5.0</max_wheel_acceleration>
       <command_topic>cmd_vel</command_topic>
       <publish_odom>true</publish_odom>
@@ -45,4 +58,6 @@
       <odometry_topic>odom</odometry_topic>
       <odometry_frame>odom</odometry_frame>
+      <!-- WORLD=1 keeps odometry in the Gazebo world coordinates used by scenarios. -->
+      <odometry_source>1</odometry_source>
       <robot_base_frame>base_footprint</robot_base_frame>
     </plugin>

Commit message: Add Ackermann route validation and streamline documentation

File: ros2_ws/src/safe_drive_description/urdf/ego_vehicle_core.xacro (robot description, xacro)
@@ -2,5 +2,5 @@
 <robot xmlns:xacro="http://www.ros.org/wiki/xacro">
   <!-- Simulator-independent geometry shared by the plain and Gazebo models. -->
-  <xacro:macro name="safe_drive_ego_vehicle" params="use_reference_mesh:=true">
+  <xacro:macro name="safe_drive_ego_vehicle" params="use_reference_mesh:=true drive_mode:=ackermann">
     <xacro:property name="chassis_length" value="4.20"/>
     <xacro:property name="chassis_width" value="1.80"/>
@@ -154,5 +154,21 @@
       </collision>
     </link>
-    <xacro:macro name="wheel" params="name x y side">
+    <xacro:macro name="wheel" params="name x y side steered:=false">
+      <xacro:if value="${steered}">
+        <link name="${name}_steering_link">
+          <inertial>
+            <mass value="0.5"/>
+            <inertia ixx="0.005" ixy="0" ixz="0" iyy="0.005" iyz="0" izz="0.005"/>
+          </inertial>
+        </link>
+        <joint name="${name}_steering_joint" type="revolute">
+          <parent link="base_link"/>
+          <child link="${name}_steering_link"/>
+          <origin xyz="${x} ${y} -0.45" rpy="0 0 0"/>
+          <axis xyz="0 0 1"/>
+          <limit lower="-0.70" upper="0.70" effort="150" velocity="1.5"/>
+          <dynamics damping="0.5" friction="0.0"/>
+        </joint>
+      </xacro:if>
       <link name="${name}">
         <inertial>
@@ -195,13 +211,15 @@
       </link>
       <joint name="${name}_joint" type="continuous">
-        <parent link="base_link"/>
+        <xacro:if value="${steered}"><parent link="${name}_steering_link"/></xacro:if>
+        <xacro:unless value="${steered}"><parent link="base_link"/></xacro:unless>
         <child link="${name}"/>
-        <origin xyz="${x} ${y} -0.45" rpy="0 0 0"/>
+        <xacro:if value="${steered}"><origin xyz="0 0 0" rpy="0 0 0"/></xacro:if>
+        <xacro:unless value="${steered}"><origin xyz="${x} ${y} -0.45" rpy="0 0 0"/></xacro:unless>
         <axis xyz="0 1 0"/>
-        <dynamics damping="0.1" friction="0.0"/>
+        <dynamics damping="${0.5 if drive_mode == 'ackermann' else 0.1}" friction="0.0"/>
       </joint>
     </xacro:macro>
-    <xacro:wheel name="front_left_wheel" x="1.25" y="0.78" side="1"/>
-    <xacro:wheel name="front_right_wheel" x="1.25" y="-0.78" side="-1"/>
+    <xacro:wheel name="front_left_wheel" x="1.25" y="0.78" side="1" steered="${drive_mode == 'ackermann'}"/>
+    <xacro:wheel name="front_right_wheel" x="1.25" y="-0.78" side="-1" steered="${drive_mode == 'ackermann'}"/>
     <xacro:wheel name="rear_left_wheel" x="-1.25" y="0.78" side="1"/>
     <xacro:wheel name="rear_right_wheel" x="-1.25" y="-0.78" side="-1"/>

File: ros2_ws/src/safe_drive_sim/urdf/ego_vehicle.gazebo.urdf.xacro (robot description, xacro)
@@ -1,12 +1,13 @@
 <?xml version="1.0"?>
 <robot name="safe_drive_ego" xmlns:xacro="http://www.ros.org/wiki/xacro">
+  <xacro:arg name="drive_mode" default="ackermann"/>
+  <xacro:property name="drive_mode" value="$(arg drive_mode)"/>
   <xacro:include filename="$(find safe_drive_description)/urdf/ego_vehicle_core.xacro"/>
-  <xacro:safe_drive_ego_vehicle/>
-  <!-- Prefer rolling in the vehicle x direction while allowing enough
-       lateral slip for stable skid-steer turns. -->
+  <xacro:safe_drive_ego_vehicle drive_mode="$(arg drive_mode)"/>
+  <!-- Steering needs lateral grip; the legacy skid-steer mode needs slip. -->
   <xacro:macro name="wheel_surface" params="name">
     <gazebo reference="${name}">
       <mu1>1.0</mu1>
-      <mu2>0.1</mu2>
+      <mu2>${1.0 if drive_mode == 'ackermann' else 0.1}</mu2>
       <fdir1>1 0 0</fdir1>
       <kp>1000000.0</kp>
@@ -33,6 +34,35 @@
     </sensor>
   </gazebo>
-  <!-- Four-wheel skid-steer drive keeps the MVP deterministic and exposes the
-       standard Twist/Odometry interface needed by the waypoint controller. -->
+  <xacro:if value="${drive_mode == 'ackermann'}">
+    <!-- This Gazebo Classic plugin reads Twist.angular.z as a tyre steering
+         angle, while linear.x is the requested forward speed. -->
+    <gazebo>
+      <plugin name="safe_drive_ackermann_drive" filename="libgazebo_ros_ackermann_drive.so">
+        <ros><namespace>/safe_drive/ego</namespace></ros>
+        <update_rate>50</update_rate>
+        <front_left_joint>front_left_wheel_joint</front_left_joint>
+        <front_right_joint>front_right_wheel_joint</front_right_joint>
+        <rear_left_joint>rear_left_wheel_joint</rear_left_joint>
+        <rear_right_joint>rear_right_wheel_joint</rear_right_joint>
+        <left_steering_joint>front_left_wheel_steering_joint</left_steering_joint>
+        <right_steering_joint>front_right_wheel_steering_joint</right_steering_joint>
+        <max_steer>0.65</max_steer>
+        <max_speed>3.0</max_speed>
+        <left_steering_pid_gain>200 0 5</left_steering_pid_gain>
+        <left_steering_i_range>0 0</left_steering_i_range>
+        <right_steering_pid_gain>200 0 5</right_steering_pid_gain>
+        <right_steering_i_range>0 0</right_steering_i_range>
+        <linear_velocity_pid_gain>100 0 1</linear_velocity_pid_gain>
+        <linear_velocity_i_range>0 0</linear_velocity_i_range>
+        <publish_odom>true</publish_odom>
+        <publish_odom_tf>true</publish_odom_tf>
+        <publish_wheel_tf>false</publish_wheel_tf>
+        <publish_steerangle>true</publish_steerangle>
+        <odometry_frame>odom</odometry_frame>
+        <robot_base_frame>base_footprint</robot_base_frame>
+      </plugin>
+    </gazebo>
+  </xacro:if>
+  <xacro:unless value="${drive_mode == 'ackermann'}">
   <gazebo>
     <plugin name="safe_drive_diff_drive" filename="libgazebo_ros_diff_drive.so">
@@ -63,3 +93,4 @@
     </plugin>
   </gazebo>
+  </xacro:unless>
 </robot>

Commit message: Stabilize traffic scene and record validation results
Tune steering, routes, signal timing, pedestrian clearance, and Gazebo startup. Save measured scenario runs and align project documentation with risk-scenario exploration as the research goal.

File: ros2_ws/src/safe_drive_description/urdf/ego_vehicle_core.xacro (robot description, xacro)
@@ -158,6 +158,6 @@
         <link name="${name}_steering_link">
           <inertial>
-            <mass value="0.5"/>
-            <inertia ixx="0.005" ixy="0" ixz="0" iyy="0.005" iyz="0" izz="0.005"/>
+            <mass value="5.0"/>
+            <inertia ixx="0.05" ixy="0" ixz="0" iyy="0.05" iyz="0" izz="0.05"/>
           </inertial>
         </link>
@@ -168,5 +168,5 @@
           <axis xyz="0 0 1"/>
           <limit lower="-0.70" upper="0.70" effort="150" velocity="1.5"/>
-          <dynamics damping="0.5" friction="0.0"/>
+          <dynamics damping="2.0" friction="0.0"/>
         </joint>
       </xacro:if>

File: ros2_ws/src/safe_drive_sim/urdf/ego_vehicle.gazebo.urdf.xacro (robot description, xacro)
@@ -49,7 +49,7 @@
         <max_steer>0.65</max_steer>
         <max_speed>21.0</max_speed>
-        <left_steering_pid_gain>200 0 5</left_steering_pid_gain>
+        <left_steering_pid_gain>500 0 20</left_steering_pid_gain>
         <left_steering_i_range>0 0</left_steering_i_range>
-        <right_steering_pid_gain>200 0 5</right_steering_pid_gain>
+        <right_steering_pid_gain>500 0 20</right_steering_pid_gain>
         <right_steering_i_range>0 0</right_steering_i_range>
         <linear_velocity_pid_gain>100 0 1</linear_velocity_pid_gain>
